Commit message: Removing old data

File: uwsim_models/uwsim_fish_urdf/Fish1.urdf (robot description, URDF)
Before this commit: robot fish1, 4 links, 3 joints
Links:
- link base_link: geometry visual mesh filename=robot/Fish1/Fish1_1_new1.obj
- link body: geometry visual mesh filename=robot/Fish1/Fish1_2_new1.obj
- link fin: geometry visual mesh filename=robot/Fish1/Fish1_Fin_new.obj
- link tail: geometry visual mesh filename=robot/Fish1/Fish1_Tail_new1.obj
Joints:
- joint Elbow: origin xyz=0 0.5 -0.3 rpy=0 0 0 -> xyz=0 0.0 -0.3 rpy=0 0 0

File: uwsim_models/uwsim_fish_urdf/Fish3.urdf (robot description, URDF)
Before this commit: robot fish3, 4 links, 3 joints
Links:
- link base_link: geometry visual mesh filename=robot/Fish3/Fish3_1_new1.obj
- link body: geometry visual mesh filename=robot/Fish3/Fish3_2_new1.obj
- link fin: geometry visual mesh filename=robot/Fish3/Fish3_fin_new1.obj
- link tail: geometry visual mesh filename=robot/Fish3/Fish3_tail_new1.obj
Joints:
- joint Slew: origin xyz=-2.3 0 0 rpy=0 0 0 -> xyz=0 0 0 rpy=0 0 0

File: uwsim_models/uwsim_fish_urdf/Fish5.urdf (robot description, URDF)
Before this commit: robot fish5, 4 links, 3 joints
Links:
- link base_link: geometry visual mesh filename=robot/Fish5/Fish5_1_new.obj
- link body: geometry visual mesh filename=robot/Fish5/Fish5_2_new.obj
- link fin: geometry visual mesh filename=robot/Fish5/Fish5_Fin_new1.obj
- link tail: geometry visual mesh filename=robot/Fish5/Fish5_Tail1_new.obj
Joints:
- joint Elbow: origin xyz=-0.5 0 2.1 rpy=0 -0.5235 0 -> xyz=-0.5 0 2.1 rpy=0 0 0
